Commit message: Add realsense

File: src/notspot_description/urdf/notspot.urdf (robot description, URDF)
Before this commit: robot notspot, 17 links, 16 joints
Links:
- added link realsense_camera_link
Joints:
- added joint realsense_camera: type fixed, parent base_link, child realsense_camera_link, origin xyz=0.13 0 0 rpy=0 0 0
